File: Omni_Rover_PCB/Battery_section.kicad_sch (KiCad schematic)
At the start: 25 parts, among them CN1 XT30PW-M, Q6 PMZ600UNEYL, Q7 PMZ600UNEYL, U26 S2B-ZR (LF)(SN), U7 BQ25303JRTER

Commit message: Finished the Laout 0 DRC ERRORS. Just needs some finishing touches.
Connections:
- net VCC renamed +5V_USB
Changed lines of the file:
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@@
 		(in_pos_files yes)
 		(dnp no)
-		(fields_autoplaced yes)
 		(property "Reference" "#PWR033"
 			(at 179.07 80.01 0)
@@
 			)
 		)
-		(property "Value" "VCC"
-			(at 179.07 71.12 0)
+		(property "Value" "+5V_USB"
+			(at 174.752 71.882 0)
 			(show_name no)
 			(do_not_autoplace no)
@@
 					(size 1.27 1.27)
 				)
+				(justify left)
 			)
 		)
