File: Omni_Rover_PCB/Power_path.kicad_sch (KiCad schematic)
At the start: 33 parts, among them Q3 JTD2302, Q4 JTD2302, Q5 JTD2302, SW3 TSA016A2526A, U1 TPS631000DRLR, U10 LM66200DRLR, U2 TPS631000DRLR

Commit message: Finished the Laout 0 DRC ERRORS. Just needs some finishing touches.
Parts:
- removed SW3: TSA016A2526A, lcsc_footprints:C2888428_SW-SMD_4P-L4_2-W3_3-P2_15-LS4_6, symbol lcsc_imported:TSA016A2526A
- added Q8: JTD2301B, lcsc_footprints:C49308281_SOT-23-3_L2_9-W1_3-P1_90-LS2_4-BR, symbol lcsc_imported:JTD2301B
- added R46, R47, R48, R49, R50: 10K, Resistor_SMD:R_0402_1005Metric_Pad0.72x0.64mm_HandSolder, symbol Device:R
- added SW6: TS1102-TD35HBM, lcsc_footprints:C36936640_SW-SMD_TS1102-TD35HBM, symbol lcsc_imported:TS1102-TD35HBM
- C27: footprint Capacitor_SMD:C_0603_1608Metric_Pad1.08x0.95mm_HandSolder -> Capacitor_SMD:C_0805_2012Metric_Pad1.18x1.45mm_HandSolder
Connections:
- net +BATT: now also Q8.2 (S), SW6.2
- net GND: now also R47.2, R48.2, R49.2, R50.2, SW6.3, SW6.4
- net at R26.2, R28.2: now also SW6.1
- net at C24.1, R23.2, R30.2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: now also Q8.1 (G)
- net TPS631000_EN renamed TPS631000_5V_EN
- net TPS631000_5V_EN: now also R50.1
- net TPS631000_MODE renamed TPS631000_3V3_MODE
- net TPS631000_3V3_MODE: now also R48.1; no longer U2.6 (MODE)
- new net: Q8.3 (D), R46.1
- new net BAT_MONITOR: R46.2, R47.1
- new net TPS631000_5V_MODE: R49.1, U2.6 (MODE)
- no-connect marks 2 -> 0
Other:
- moved on the sheet: C1, C2, C24, C25, C26, C27, C28, C3, C4, L1, L2, Q3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
