File: Omni_Rover_PCB/Omni_Rover_PCB.kicad_pcb (KiCad board)
At the start: 2 copper layers, 160 parts, among them CN1 XT30PW-M, CN2 1.0-6PWT, J1 Conn_01x04_Socket, J2 USB_C_Receptacle_USB2.0_16P, Q1 SS8050, Q2 SS8050, Q3 JTD2302, Q4 JTD2302, Q5 JTD2302, Q6 PMZ600UNEYL, Q7 PMZ600UNEYL, SW1 TSA016A2526A, SW2 TSA016A2526A, SW3 TSA016A2526A, U1 TPS631000DRLR, U10 LM66200DRLR, U11 XL-1010RGBC-WS2812B, U12 XL-1010RGBC-WS2812B, U13 XL-1010RGBC-WS2812B, U14 XL-1010RGBC-WS2812B, U15 XL-1010RGBC-WS2812B, U16 XL-1010RGBC-WS2812B, U17 XL-1010RGBC-WS2812B, U18 XL-1010RGBC-WS2812B, U19 XL-1010RGBC-WS2812B, U2 TPS631000DRLR, U20 XL-1010RGBC-WS2812B, U21 XL-1010RGBC-WS2812B, U22 XL-1010RGBC-WS2812B, U23 XL-1010RGBC-WS2812B, U24 XL-1010RGBC-WS2812B, U25 XL-1010RGBC-WS2812B, U26 S2B-ZR (LF)(SN), U27 S2B-ZR (LF)(SN), U28 DRV8837DSGR, U29 S2B-ZR (LF)(SN), U3 CH340C, U30 DRV8837DSGR, U31 S2B-ZR (LF)(SN), U32 DRV8837DSGR, U33 S2B-ZR (LF)(SN), U4 ESP32-WROOM-32D, U5 USBLC6-2SC6, U6 DRV8837DSGR, U7 BQ25303JRTER, U8 SN74LV1T34DCK, U9 XL-1010RGBC-WS2812B

Commit message: Finished the Laout 0 DRC ERRORS. Just needs some finishing touches.
Parts:
- removed SW3: TSA016A2526A, lcsc_footprints:C2888428_SW-SMD_4P-L4_2-W3_3-P2_15-LS4_6
- added C61: 100nF, Capacitor_SMD:C_0402_1005Metric_Pad0.74x0.62mm_HandSolder, F.Cu at (145.7, 104.0)
- added C62: 2.2uF, Capacitor_SMD:C_0402_1005Metric_Pad0.74x0.62mm_HandSolder, F.Cu at (146.9, 104.0)
- added C63: 100nF, Capacitor_SMD:C_0402_1005Metric_Pad0.74x0.62mm_HandSolder, F.Cu at (148.8, 107.5)
- added C64: 100nF, Capacitor_SMD:C_0402_1005Metric_Pad0.74x0.62mm_HandSolder, F.Cu at (143.6, 104.7)
- added C65: 100nF, Capacitor_SMD:C_0402_1005Metric_Pad0.74x0.62mm_HandSolder, F.Cu at (183.9, 85.5)
- added C66: 100nF, Capacitor_SMD:C_0402_1005Metric_Pad0.74x0.62mm_HandSolder, F.Cu at (183.9, 92.5)
- added H1: MountingHole_Pad, MountingHole:MountingHole_3.2mm_M3_Pad_Via, F.Cu at (118.0, 68.5)
- added H2: MountingHole_Pad, MountingHole:MountingHole_3.2mm_M3_Pad_Via, F.Cu at (168.0, 68.5)
- added H3: MountingHole_Pad, MountingHole:MountingHole_3.2mm_M3_Pad_Via, F.Cu at (118.0, 138.6)
- added H4: MountingHole_Pad, MountingHole:MountingHole_3.2mm_M3_Pad_Via, F.Cu at (168.0, 138.6)
- added H5: MountingHole_Pad, MountingHole:MountingHole_3.2mm_M3_Pad_Via, F.Cu at (185.5, 105.8)
- added Q8: JTD2301B, lcsc_footprints:C49308281_SOT-23-3_L2_9-W1_3-P1_90-LS2_4-BR, F.Cu at (162.4, 126.0)
- added R41: 10K, Resistor_SMD:R_0402_1005Metric_Pad0.72x0.64mm_HandSolder, F.Cu at (146.6, 101.0)
- added R42: 10K, Resistor_SMD:R_0402_1005Metric_Pad0.72x0.64mm_HandSolder, F.Cu at (140.0, 102.5)
- added R43: 4.7K, Resistor_SMD:R_0402_1005Metric_Pad0.72x0.64mm_HandSolder, F.Cu at (104.7, 89.0)
- added R44: 4.7K, Resistor_SMD:R_0402_1005Metric_Pad0.72x0.64mm_HandSolder, F.Cu at (107.4, 89.0)
- added R45: 0R, Resistor_SMD:R_0402_1005Metric_Pad0.72x0.64mm_HandSolder, F.Cu at (120.8, 105.7)
- added R46: 10K, Resistor_SMD:R_0402_1005Metric_Pad0.72x0.64mm_HandSolder, F.Cu at (160.6, 70.2)
- added R47: 10K, Resistor_SMD:R_0402_1005Metric_Pad0.72x0.64mm_HandSolder, F.Cu at (160.6, 67.2)
- added R48: 10K, Resistor_SMD:R_0402_1005Metric_Pad0.72x0.64mm_HandSolder, F.Cu at (117.0, 119.5)
- added R49: 10K, Resistor_SMD:R_0402_1005Metric_Pad0.72x0.64mm_HandSolder, F.Cu at (141.8, 110.1)
- added R50: 10K, Resistor_SMD:R_0402_1005Metric_Pad0.72x0.64mm_HandSolder, F.Cu at (139.7, 115.7)
- added R51: 100K, Resistor_SMD:R_0402_1005Metric_Pad0.72x0.64mm_HandSolder, F.Cu at (182.4, 81.7)
- added R52: 10K, Resistor_SMD:R_0402_1005Metric_Pad0.72x0.64mm_HandSolder, F.Cu at (184.6, 83.5)
- added R53: 100K, Resistor_SMD:R_0402_1005Metric_Pad0.72x0.64mm_HandSolder, F.Cu at (182.4, 88.6)
- added R54: 10K, Resistor_SMD:R_0402_1005Metric_Pad0.72x0.64mm_HandSolder, F.Cu at (184.6, 90.5)
- added SW4: TS1102-TD35HBM, lcsc_footprints:C36936640_SW-SMD_TS1102-TD35HBM, F.Cu at (188.0, 85.2)
- added SW5: TS1102-TD35HBM, lcsc_footprints:C36936640_SW-SMD_TS1102-TD35HBM, F.Cu at (188.0, 92.2)
- added SW6: TS1102-TD35HBM, lcsc_footprints:C36936640_SW-SMD_TS1102-TD35HBM, F.Cu at (188.0, 99.2)
- added U34: TCA9555PWR, Package_SO:TSSOP-24_4.4x7.8mm_P0.65mm, F.Cu at (146.6, 112.3)
- added U35: LSM6DS3, Package_LGA:LGA-14_3x2.5mm_P0.5mm_LayoutBorder3x4y, F.Cu at (143.1, 102.4)
- added kobee-studio-6AB2BFE9: Kobee Studio, kobee-studio-6AB2BF39, F.Cu at (143.4, 82.9)
- C27: footprint Capacitor_SMD:C_0603_1608Metric_Pad1.08x0.95mm_HandSolder -> Capacitor_SMD:C_0805_2012Metric_Pad1.18x1.45mm_HandSolder
- C44, C45, C46, C47, CN2, U26: moved to B.Cu
- moved C23 1203.7 mm to (145.9, 76.3)
- moved C29 1203.7 mm to (143.4, 76.3)
- moved C30 1203.7 mm to (140.9, 76.3)
- moved C31 1203.7 mm to (138.4, 76.3)
- moved C32 1203.7 mm to (138.4, 78.8)
- moved C33 1203.7 mm to (140.9, 78.8)
- moved C34 1203.7 mm to (143.4, 78.8)
- moved C35 1203.7 mm to (145.9, 78.8)
- moved C36 1203.7 mm to (145.9, 81.3)
- moved C37 1203.7 mm to (143.4, 81.3)
- moved C38 1203.7 mm to (140.9, 81.3)
- moved C39 1203.7 mm to (138.4, 81.3)
- moved C40 1203.7 mm to (138.4, 83.8)
- moved C41 1203.7 mm to (140.9, 83.8)
- moved C42 1203.7 mm to (143.4, 83.8)
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Connections:
- net /Battery_section/BQ25303J_EN renamed /P7
- net /Motor_drivers/SLEEP renamed /P15
- net /Power_path/LM66200_ST renamed /P11
- C19 pad 1: VCC -> +5V_USB
- J2 pad A5: /CC1 -> /ESP32/I39
- J2 pad B5: /CC2 -> /ESP32/I34
- Q5 pad 3: /Power_path/ON_SW -> /ESP32/I36
- R14 pad 1: /CC2 -> /ESP32/I34
- R15 pad 1: /CC1 -> /ESP32/I39
- R29 pad 2: /Power_path/ON_SW -> /ESP32/I36
- R31 pad 1: /Power_path/TURN_ON -> /ESP32/IO27
- R39 pad 1: /Battery_section/1A_CHRG -> /P5
- R40 pad 1: /Battery_section/2A_CHRG -> /P6
- U1 pad 6: /Power_path/TPS631000_MODE -> /P10
- U2 pad 5: /Power_path/TPS631000_EN -> /P1
- U2 pad 6: /Power_path/TPS631000_MODE -> /P0
- U28 pad 5: /Motor_drivers/RU_2 -> /ESP32/IO18
- U28 pad 6: /Motor_drivers/RU_1 -> /ESP32/IO17
- U3 pad 5: /ESP32/D+ -> /USB.D+
- U3 pad 6: /ESP32/D- -> /USB.D-
- U30 pad 5: /Motor_drivers/LL_2 -> /ESP32/IO33
- U30 pad 6: /Motor_drivers/LL_1 -> /ESP32/IO32
- U32 pad 5: /Motor_drivers/RL_2 -> /ESP32/IO26
- U32 pad 6: /Motor_drivers/RL_1 -> /ESP32/IO25
- U4 pad 10: /ESP32/GPIO25 -> /ESP32/IO25
- U4 pad 11: /ESP32/GPIO26 -> /ESP32/IO26
- U4 pad 12: /ESP32/GPIO27 -> /ESP32/IO27
- U4 pad 16: /ESP32/GPIO13 -> Net-(U4-IO13)
- U4 pad 27: /ESP32/GPIO16 -> /ESP32/IO16
- U4 pad 28: /ESP32/GPIO17 -> /ESP32/IO17
- U4 pad 30: /ESP32/GPIO18 -> /ESP32/IO18
- U4 pad 31: /ESP32/GPIO19 -> /ESP32/IO19
- U4 pad 33: /ESP32/GPIO21 -> /ESP32/IO21
- U4 pad 36: /ESP32/GPIO22 -> /ESP32/IO22
- U4 pad 37: /ESP32/GPIO23 -> /ESP32/IO23
- U4 pad 4: /ESP32/GPIO36 -> /ESP32/I36
- U4 pad 5: /ESP32/GPIO39 -> /ESP32/I39
- U4 pad 6: /ESP32/GPIO34 -> /ESP32/I34
- U4 pad 7: /ESP32/GPIO35 -> /ESP32/I35
- U4 pad 8: /ESP32/GPIO32 -> /ESP32/IO32
- U4 pad 9: /ESP32/GPIO33 -> /ESP32/IO33
- U5 pad 4: /USB_D+ -> /USB.D+
- U5 pad 6: /USB_D_ -> /USB.D-
- U6 pad 5: /Motor_drivers/LU_2 -> /ESP32/IO23
- U6 pad 6: /Motor_drivers/LU_1 -> /ESP32/IO19
- U7 pad 1: VCC -> +5V_USB
- U8 pad 2: /LED_section/LED_DIN -> /ESP32/IO16
Routing:
- net +3V3: track 30.3 -> 428.8 mm, vias 12 -> 17
- net /P15: track 0.00 -> 289.2 mm, vias 0 -> 7
- net /ESP32/I39: track 0.00 -> 173.2 mm, vias 0 -> 10
- net /ESP32/I34: track 0.00 -> 160.7 mm, vias 0 -> 9
- net /ESP32/IO25: track 0.00 -> 121.1 mm, vias 0 -> 2
- net /ESP32/IO26: track 0.00 -> 117.8 mm, vias 0 -> 2
- net /ESP32/I36: track 0.00 -> 97.9 mm, vias 0 -> 4
- net /ESP32/I35: track 0.00 -> 84.6 mm, vias 0 -> 4
- net /ESP32/IO18: track 0.00 -> 74.4 mm, vias 0 -> 2
- net /ESP32/IO17: track 0.00 -> 73.1 mm, vias 0 -> 2
- net /USB.D-: track 0.00 -> 71.4 mm, vias 0 -> 6
- net /USB.D+: track 0.00 -> 68.6 mm, vias 0 -> 6
- net /ESP32/IO22: track 0.00 -> 64.2 mm, vias 0 -> 5
- net /P10: track 0.00 -> 62.4 mm, vias 0 -> 2
- net Net-(Q8-D): track 0.00 -> 58.0 mm
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- added copper zone on B.Cu, net +5V
- added copper zone on B.Cu, net +5V_USB
- added copper zone on F.Cu, net +5V_USB
- added copper zone on B.Cu, net +BATT
- added copper zone on B.Cu, net GND
- removed copper zone on F.Cu, net VCC
Other:
- board outline added: 100 x 100 mm
- board text added: "BATTERY"
- board text removed: "Battery_section"
- board text removed: "ESP32"
- board text removed: "LED_section"
- board text removed: "Main Sheet"
- board text removed: "Motor_drivers"
- board text removed: "Power_path"

Commit message: Made soem minor fixes to the schematic and PCB layout.
Parts:
- removed kibuzzard-6AAEA8E7: G***, kibuzzard-6AAEA8E7
- added C67: 22uF, Capacitor_SMD:C_0805_2012Metric_Pad1.18x1.45mm_HandSolder, F.Cu at (103.0, 121.2)
- added kobee-studio-6AB59811: Kobee Studio, kobee-studio-6AB59747, F.Cu at (181.5, 99.2)
- added kobee-studio-6AB59858: Kobee Studio, kobee-studio-6AB59747, F.Cu at (172.8, 92.5)
- added kobee-studio-6AB59875: Kobee Studio, kobee-studio-6AB59747, F.Cu at (173.5, 85.3)
- added kobee-studio-6AB598B2: Kobee Studio, kobee-studio-6AB598B2, F.Cu at (189.7, 109.5)
- added kobee-studio-6AB598D9: Kobee Studio, kobee-studio-6AB598D9, F.Cu at (150.2, 149.4)
- added kobee-studio-6AB598D9: Kobee Studio, kobee-studio-6AB598D9, B.Cu at (150.2, 149.4)
- added kobee-studio-6AB59952: Kobee Studio, kobee-studio-6AB598D9, F.Cu at (135.4, 149.4)
- added kobee-studio-6AB59952: Kobee Studio, kobee-studio-6AB598D9, B.Cu at (135.4, 149.4)
- added kobee-studio-6AB59AC1: Kobee Studio, kobee-studio-6AB59681, F.Cu at (102.5, 84.6)
- added kobee-studio-6AB5A115: Kobee Studio, kobee-studio-6AB5A115, F.Cu at (164.8, 96.4)
- added kobee-studio-6AB5A152: Kobee Studio, kobee-studio-6AB5A14C, F.Cu at (161.6, 96.4)
- added kobee-studio-6AB5A28E: Kobee Studio, kobee-studio-6AB5A211, B.Cu at (126.1, 87.2)
- added kobee-studio-6AB5A2B4: Kobee Studio, kobee-studio-6AB5A2B4, B.Cu at (130.8, 145.9)
- moved kobee-studio-6AADB37A 1.39 mm to (123.2, 123.5)
- moved J1 1.22 mm to (102.5, 84.8)
- moved R33 1.21 mm to (117.2, 121.5)
- moved R43 0.65 mm to (104.0, 89.0)
Routing:
- net Net-(U1-VIN): track 5.90 -> 3.06 mm
- net +3V3: track 428.8 -> 430.1 mm, vias 17 -> 19
- net /ESP32/TX_ESP: track 47.5 -> 46.1 mm
- net Net-(U1-EN): track 3.12 -> 4.38 mm
- net /ESP32/RX_ESP: track 46.3 -> 45.3 mm
- net GND: vias 309 -> 547
- net +BATT: vias 82 -> 86
